File: ft601.kicad_sch (KiCad schematic)
At the start: 36 parts, among them J2 Conn_02x26, J3 Conn_01x03, J4 Conn_01x03, J5 Conn_01x04, J6 Conn_01x04, U1 FT601Q, Y2 X322530MOB4SI

Commit message: JLCPCB order. W2026020708395445
Parts:
- removed RN1, RN10, RN11, RN2, RN3, RN4, RN5, RN6, RN7, RN8, RN9: 33R, SamaSys_Parts:EXB28V510JX, symbol Device:R_Pack04
- added R32, R33, R34, R35, R36, R37, R38, R39: 33R, Resistor_SMD:R_0603_1608Metric, symbol Device:R
Connections:
- net BE_0: now also U1.4 (BE_0)
- net BE_1: now also U1.5 (BE_1)
- net BE_2: now also U1.6 (BE_2)
- net BE_3: now also U1.7 (BE_3)
- net D0: now also U1.40 (DATA_0)
- net D1: now also U1.41 (DATA_1)
- net D10: now also U1.52 (DATA_10)
- net D11: now also U1.53 (DATA_11)
- net D12: now also U1.54 (DATA_12)
- net D13: now also U1.55 (DATA_13)
- net D14: now also U1.56 (DATA_14)
- net D15: now also U1.57 (DATA_15)
- net D16: now also U1.60 (DATA_16)
- net D17: now also U1.61 (DATA_17)
- net D18: now also U1.62 (DATA_18)
- net D19: now also U1.63 (DATA_19)
- net D2: now also U1.42 (DATA_2)
- net D20: now also U1.64 (DATA_20)
- net D21: now also U1.65 (DATA_21)
- net D22: now also U1.66 (DATA_22)
- net D23: now also U1.67 (DATA_23)
- net D24: now also U1.69 (DATA_24)
- net D25: now also U1.70 (DATA_25)
- net D26: now also U1.71 (DATA_26)
- net D27: now also U1.72 (DATA_27)
- net D28: now also U1.73 (DATA_28)
- net D29: now also U1.74 (DATA_29)
- net D3: now also U1.43 (DATA_3)
- net D30: now also U1.75 (DATA_30)
- net D31: now also U1.76 (DATA_31)
- net D4: now also U1.44 (DATA_4)
- net D5: now also U1.45 (DATA_5)
- net D6: now also U1.46 (DATA_6)
- net D7: now also U1.47 (DATA_7)
- net D8: now also U1.50 (DATA_8)
- net D9: now also U1.51 (DATA_9)
- net GND: now also R32.2, R33.2
- net SIWU_N: now also R37.1
- net WR_N: now also R36.1
- net at J6.1 (Pin_1): now also R32.1
- net at J6.2 (Pin_2): now also R33.1
- net at J6.3 (Pin_3): now also R34.1
- net at J6.4 (Pin_4): now also R35.1
- net at J5.1 (Pin_1): now also R36.2
- net at J5.2 (Pin_2): now also R37.2
- net at J5.3 (Pin_3): now also R38.2
- net at J5.4 (Pin_4): now also R39.2
- net at U1.13 (~{OE}): now also R34.2
- net at U1.12 (~{RD}): now also R35.2
- net at U1.8 (~{TXE}): now also R39.1
- net at U1.9 (~{RXF}): now also R38.1
