File: ft601_module.kicad_pcb (KiCad board)
At the start: 4 copper layers, 62.7 x 67.6 mm, 99 parts, among them IC1 HD3SS3220IRNHR, IC2 TLV75510PDBVR, IC3 TLV75533PDBVR, J1 Conn_01x02, J2 Conn_02x26, J3 Conn_01x03, J4 Conn_01x03, J5 Conn_01x04, J6 Conn_01x04, J7 12401598E4-2A, J8 Conn_01x02, J9 Conn_01x03, U1 FT601Q, U2 TPD6E05U06RVZR, U3 TPD4E05U06DQAR, U4 TPD4E05U06DQAR, Y2 X322530MOB4SI

Commit message: JLCPCB order. W2026020708395445
Parts:
- removed RN1, RN10, RN11, RN2, RN3, RN4, RN5, RN6, RN7, RN8, RN9: 33R, SamaSys_Parts:EXB28V510JX
- added R32: 33R, Resistor_SMD:R_0603_1608Metric, F.Cu at (160.8, 80.6)
- added R33: 33R, Resistor_SMD:R_0603_1608Metric, F.Cu at (161.6, 83.6)
- added R34: 33R, Resistor_SMD:R_0603_1608Metric, F.Cu at (162.4, 80.6)
- added R35: 33R, Resistor_SMD:R_0603_1608Metric, F.Cu at (163.3, 83.6)
- added R36: 33R, Resistor_SMD:R_0603_1608Metric, F.Cu at (164.6, 80.6)
- added R37: 33R, Resistor_SMD:R_0603_1608Metric, F.Cu at (165.3, 83.6)
- added R38: 33R, Resistor_SMD:R_0603_1608Metric, F.Cu at (166.2, 80.6)
- added R39: 33R, Resistor_SMD:R_0603_1608Metric, F.Cu at (166.9, 83.6)
- FB1, FB2, FB3: value HI1206N101R-00 -> GZ1608D601TF; footprint SamaSys_Parts:BEADC3216X130N -> SamaSys_Parts:BEADC1608X95N
- moved FB1 5.93 mm to (135.0, 75.8), turned to 0 degrees
- moved FB3 3.36 mm to (139.6, 75.3), turned to 180 degrees
- moved FB2 2.44 mm to (136.9, 78.1), turned to 90 degrees
- moved C23 0.90 mm to (138.3, 71.8), turned to 90 degrees
- moved J9 0.75 mm to (124.6, 69.0)
- moved R25 0.40 mm to (137.3, 64.7)
- moved J4 0.39 mm to (134.7, 61.4)
- moved J8 0.29 mm to (124.6, 61.4)
- moved J3 0.11 mm to (144.9, 61.4)
- moved J6 0.08 mm to (155.1, 61.4)
- moved J5 0.07 mm to (167.8, 61.4)
Connections:
- FB1 pad 1: PLL_AVDD -> +3.3V
- FB1 pad 2: VD10 -> VCC33
- FB2 pad 1: +3.3V -> VCC33
- FB2 pad 2: VCC33 -> VCCIO
- FB3 pad 1: VCC33 -> PLL_AVDD
- FB3 pad 2: VCCIO -> VD10
- U1 pad 4: Net-(RN5-R1.2) -> /ft601/BE_0
- U1 pad 40: Net-(RN1-R1.2) -> /ft601/D0
- U1 pad 41: Net-(RN1-R2.2) -> /ft601/D1
- U1 pad 42: Net-(RN1-R3.2) -> /ft601/D2
- U1 pad 43: Net-(RN1-R4.2) -> /ft601/D3
- U1 pad 44: Net-(RN2-R1.2) -> /ft601/D4
- U1 pad 45: Net-(RN2-R2.2) -> /ft601/D5
- U1 pad 46: Net-(RN2-R3.2) -> /ft601/D6
- U1 pad 47: Net-(RN2-R4.2) -> /ft601/D7
- U1 pad 5: Net-(RN5-R2.2) -> /ft601/BE_1
- U1 pad 50: Net-(RN3-R1.2) -> /ft601/D8
- U1 pad 51: Net-(RN3-R2.2) -> /ft601/D9
- U1 pad 52: Net-(RN3-R3.2) -> /ft601/D10
- U1 pad 53: Net-(RN3-R4.2) -> /ft601/D11
- U1 pad 54: Net-(RN4-R1.2) -> /ft601/D12
- U1 pad 55: Net-(RN4-R2.2) -> /ft601/D13
- U1 pad 56: Net-(RN4-R3.2) -> /ft601/D14
- U1 pad 57: Net-(RN4-R4.2) -> /ft601/D15
- U1 pad 6: Net-(RN5-R3.2) -> /ft601/BE_2
- U1 pad 60: Net-(RN8-R1.2) -> /ft601/D16
- U1 pad 61: Net-(RN8-R2.2) -> /ft601/D17
- U1 pad 62: Net-(RN8-R3.2) -> /ft601/D18
- U1 pad 63: Net-(RN8-R4.2) -> /ft601/D19
- U1 pad 64: Net-(RN9-R1.2) -> /ft601/D20
- U1 pad 65: Net-(RN9-R2.2) -> /ft601/D21
- U1 pad 66: Net-(RN9-R3.2) -> /ft601/D22
- U1 pad 67: Net-(RN9-R4.2) -> /ft601/D23
- U1 pad 69: Net-(RN10-R1.2) -> /ft601/D24
- U1 pad 7: Net-(RN5-R4.2) -> /ft601/BE_3
- U1 pad 70: Net-(RN10-R2.2) -> /ft601/D25
- U1 pad 71: Net-(RN10-R3.2) -> /ft601/D26
- U1 pad 72: Net-(RN10-R4.2) -> /ft601/D27
- U1 pad 73: Net-(RN11-R1.2) -> /ft601/D28
- U1 pad 74: Net-(RN11-R2.2) -> /ft601/D29
- U1 pad 75: Net-(RN11-R3.2) -> /ft601/D30
- U1 pad 76: Net-(RN11-R4.2) -> /ft601/D31
Routing:
- net /ft601/D0: track 3.79 -> 33.2 mm
- net /ft601/D1: track 6.12 -> 34.7 mm
- net Net-(RN1-R1.2): track 28.2 -> 0.00 mm
- net /ft601/D2: track 3.48 -> 31.2 mm
- net Net-(RN1-R2.2): track 27.6 -> 0.00 mm
- net /ft601/D3: track 8.33 -> 35.3 mm
- net Net-(RN1-R3.2): track 26.9 -> 0.00 mm
- net Net-(RN1-R4.2): track 26.1 -> 0.00 mm
- net /ft601/D4: track 3.29 -> 28.3 mm
- net /ft601/D5: track 6.09 -> 30.3 mm
- net Net-(RN2-R1.2): track 23.8 -> 0.00 mm
- net /ft601/D6: track 3.90 -> 27.4 mm
- net Net-(RN2-R2.2): track 23.3 -> 0.00 mm
- net /ft601/D7: track 6.64 -> 29.3 mm
- net Net-(RN2-R3.2): track 22.6 -> 0.00 mm
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