File: power.kicad_sch (KiCad schematic)
At the start: 31 parts, among them IC2 TLV75510PDBVR, IC3 TLV75533PDBVR, J8 Conn_01x02, J9 Conn_01x03

Commit message: JLCPCB order. W2026020708395445
Parts:
- removed FB1, FB2, FB3: HI1206N101R-00, SamaSys_Parts:BEADC3216X130N, symbol SamacSys_Parts:HI1206N101R-00
- added FB1, FB2, FB3: GZ1608D601TF, SamaSys_Parts:BEADC1608X95N, symbol SamacSys_Parts:GZ1608D601TF
Connections:
- net +3.3V: now also FB1.1
- net PLL_AVDD: now also FB3.1
- net VCC33: now also FB1.2, FB2.1
- net VCCIO: now also FB2.2
- net VD10: now also FB3.2
